Commit message: 5dof tensegrity robot with linear base and robotiq gripper
Fixes #19

File: res/Tensegrity/urdf/threedof_manipulator.urdf (robot description, URDF)
Before this commit: robot threedof_manipulator, 7 links, 6 joints
Links:
- removed link Endeffektor_x
- removed link Endeffektor_y
- removed link Mesh_Endeffektor
- removed link Mesh_Unterarm
- removed link Oberarm
- removed link Unterarm
- removed link world
- added link cylinder_approx_link, mass 0.192; collision cylinder length=0.02 radius=0.083; visual cylinder length=0.02 radius=0.083
- added link end_effector_link, mass 0.4; collision mesh filename=/home/robot/studentische-arbeiten/res/Tensegrity/meshes/End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 scale=0.001 0.001 0.001; visual mesh filename=/home/robot/studentische-arbeiten/res/Tensegrity/meshes/End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 scale=0.001 0.001 0.001
- added link forearm_link, mass 1.9; collision mesh filename=/home/robot/studentische-arbeiten/res/Tensegrity/meshes/Unt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 scale=0.001 0.001 0.001; visual mesh filename=/home/robot/studentische-arbeiten/res/Tensegrity/meshes/Unt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 scale=0.001 0.001 0.001
- added link root_link, mass 0.0001
- added link tool_link, mass 0.0001
- added link upper_arm_link, mass 2; collision mesh filename=/home/robot/studentische-arbeiten/res/Tensegrity/meshes/Obe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 scale=0.001 0.001 0.001; visual mesh filename=/home/robot/studentische-arbeiten/res/Tensegrity/meshes/Obe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 scale=0.001 0.001 0.001
- added link wrist_x_link, mass 0.0001; collision sphere radius=0.005; visual sphere radius=0.005
- added link wrist_y_link, mass 0.0001; collision sphere radius=0.005; visual sphere radius=0.005
Joints:
- removed joint Joint1
- removed joint Rahmen_Oberarm
- removed joint Wrist_Joint_x
- removed joint Wrist_Joint_y
- removed joint cylinder1_Unterarm
- removed joint fixed_Wrist_Mesh
- added joint cylinder_forearm_fixed_joint: type fixed, parent cylinder_approx_link, child forearm_link, origin xyz=0.193 0 0 rpy=1.57 3.14 -1.57
- added joint ee_tool_fixed_joint: type fixed, parent end_effector_link, child tool_link, origin xyz=0 0 0.11768 rpy=0 0 0
- added joint elbow_joint: type revolute, parent upper_arm_link, child cylinder_approx_link, origin xyz=0.352 0.0226 0 rpy=1.57 0 0, axis 0 0 1, limit lower=-1.5 upper=1.5 effort=0.125 velocity=1.0
- added joint root_upper_arm_fixed_joint: type fixed, parent root_link, child upper_arm_link, origin xyz=-0.0225 0.007 -0.10244 rpy=1.57 1.57 0
- added joint wrist_mesh_fixed_joint: type fixed, parent wrist_x_link, child end_effector_link, origin xyz=0 0 -0.0033 rpy=3.14 0 2.616
- added joint wrist_x_joint: type revolute, parent wrist_y_link, child wrist_x_link, origin xyz=0 0 0 rpy=0 0 0, axis 0 1 0, limit lower=-0.8 upper=0.8 effort=10.0 velocity=0.5
- added joint wrist_y_joint: type revolute, parent forearm_link, child wrist_y_link, origin xyz=0 0 -0.241 rpy=0 0 3.14, axis 1 0 0, limit lower=-0.8 upper=0.8 effort=10.0 velocity=0.5
