Commit message: Remodeled tensegrity wrist meshes + pipeline skript

File: res/Tensegrity/deprecated/urdf/twodof_wrist_mini.urdf (robot description, URDF)
Before this commit: robot twodof_wrist, 4 links, 3 joints
Joints:
- joint wrist_x_joint: origin xyz=0 0 -0.042 rpy=0 0 3.14 -> xyz=0 0 -0.046 rpy=0 0 3.14
